File: zaehlerboard/zaehlerboard.sch (KiCad schematic (older format))
At the start: 10 parts, among them Q1 Q_Photo_NPN, U1 TL084

Commit message: updated circuit
Parts:
- removed D2: LED, symbol Device:LED
- removed R5: 68, symbol Device:R
- removed V?: 5V, symbol pspice:VSOURCE
- added R?: R, symbol Device:R
- U1: value TL084 -> LM293
Connections:
- wire segments 24 -> 18
- no-connect marks 0 -> 1
Other:
- moved on the sheet: RV?
Changed lines of the file:
@@
 EESchema Schematic File Version 4
-EELAYER 29 0
+LIBS:zaehlerboard-cache
+EELAYER 30 0
 EELAYER END
 $Descr A4 11693 8268
@@
 P 7450 3050
 F 0 "U1" H 7450 2683 50  0000 C CNN
-F 1 "TL084" H 7450 2774 50  0000 C CNN
+F 1 "LM293" H 7450 2774 50  0000 C CNN
 F 2 "" H 7400 3150 50  0001 C CNN
 F 3 "http://www.ti.com/lit/ds/symlink/tl081.pdf" H 7500 3250 50  0001 C CNN
@@
 	6450 2550 6450 2400
 $Comp
-L Device:LED D2
-U 1 1 5D3787A5
-P 8050 3250
-F 0 "D2" V 7997 3328 50  0000 L CNN
-F 1 "LED" V 8088 3328 50  0000 L CNN
-F 2 "" H 8050 3250 50  0001 C CNN
-F 3 "~" H 8050 3250 50  0001 C CNN
-	1    8050 3250
-	0    1    1    0
-$EndComp
-Wire Wire Line
-	8050 3100 8050 3050
-Wire Wire Line
-	8050 3050 7750 3050
-$Comp
-L power:GND #PWR0106
-U 1 1 5D37A511
-P 8050 3850
-F 0 "#PWR0106" H 8050 3600 50  0001 C CNN
-F 1 "GND" H 8055 3677 50  0000 C CNN
-F 2 "" H 8050 3850 50  0001 C CNN
-F 3 "" H 8050 3850 50  0001 C CNN
-	1    8050 3850
-	1    0    0    -1
-$EndComp
-Wire Wire Line
-	8050 3400 8050 3450
-$Comp
 L power:GND #PWR0107
 U 1 1 5D37E686
@@
 	1    0    0    -1
 $EndComp
-$Comp
-L Device:R R5
-U 1 1 5D383A13
-P 8050 3600
-F 0 "R5" H 8120 3646 50  0000 L CNN
-F 1 "68" H 8120 3555 50  0000 L CNN
-F 2 "" V 7980 3600 50  0001 C CNN
-F 3 "~" H 8050 3600 50  0001 C CNN
-	1    8050 3600
-	1    0    0    -1
-$EndComp
-Wire Wire Line
-	8050 3750 8050 3850
 Wire Wire Line
 	4700 3500 4700 3850
@@
 L Device:R_POT RV?
 U 1 1 5D39FFBD
-P 7100 2550
-F 0 "RV?" V 6893 2550 50  0000 C CNN
-F 1 "10k" V 6984 2550 50  0000 C CNN
-F 2 "" H 7100 2550 50  0001 C CNN
-F 3 "~" H 7100 2550 50  0001 C CNN
-	1    7100 2550
+P 7000 2550
+F 0 "RV?" V 6793 2550 50  0000 C CNN
+F 1 "10k" V 6884 2550 50  0000 C CNN
+F 2 "" H 7000 2550 50  0001 C CNN
+F 3 "~" H 7000 2550 50  0001 C CNN
+	1    7000 2550
 	0    -1   1    0
 $EndComp
-$Comp
-L pspice:VSOURCE V?
-U 1 1 5D3A4C6A
-P 2300 3300
-F 0 "V?" H 2528 3346 50  0000 L CNN
-F 1 "5V" H 2528 3255 50  0000 L CNN
-F 2 "" H 2300 3300 50  0001 C CNN
-F 3 "~" H 2300 3300 50  0001 C CNN
-	1    2300 3300
-	1    0    0    -1
-$EndComp
-$Comp
-L power:GND #PWR?
-U 1 1 5D3A5546
-P 2300 3800
-F 0 "#PWR?" H 2300 3550 50  0001 C CNN
-F 1 "GND" H 2305 3627 50  0000 C CNN
-F 2 "" H 2300 3800 50  0001 C CNN
-F 3 "" H 2300 3800 50  0001 C CNN
-	1    2300 3800
-	1    0    0    -1
-$EndComp
-$Comp
-L power:VCC #PWR?
-U 1 1 5D3A5CE5
-P 2300 2750
-F 0 "#PWR?" H 2300 2600 50  0001 C CNN
-F 1 "VCC" H 2317 2923 50  0000 C CNN
-F 2 "" H 2300 2750 50  0001 C CNN
-F 3 "" H 2300 2750 50  0001 C CNN
-	1    2300 2750
-	1    0    0    -1
-$EndComp
-Wire Wire Line
-	2300 3000 2300 2750
-Wire Wire Line
-	2300 3600 2300 3800
-Wire Wire Line
-	7250 2550 7650 2550
-Wire Wire Line
-	6450 2550 6950 2550
-Wire Wire Line
-	7100 2700 7100 2800
-Wire Wire Line
-	7100 2800 7000 2800
-Wire Wire Line
-	7000 2800 7000 2950
+Wire Wire Line
+	6450 2550 6850 2550
+$Comp
+L Device:R R?
+U 1 1 5D47120C
+P 8350 2900
+F 0 "R?" H 8420 2946 50  0000 L CNN
+F 1 "R" H 8420 2855 50  0000 L CNN
+F 2 "" V 8280 2900 50  0001 C CNN
+F 3 "~" H 8350 2900 50  0001 C CNN
+	1    8350 2900
+	1    0    0    -1
+$EndComp
+Wire Wire Line
+	7750 3050 8350 3050
+Connection ~ 6850 2550
+Wire Wire Line
+	6850 2550 6950 2550
+Wire Wire Line
+	7000 2700 7000 2950
+NoConn ~ 7750 3650
+Wire Wire Line
+	7150 2550 7650 2550
 $EndSCHEMATC
