File: zaehlerboard/zaehlerboard.kicad_pcb (KiCad board)
At the start: 2 copper layers, 0 parts

Commit message: update circuit
Parts:
- added C1: 100nF, Capacitor_THT:C_Disc_D5.0mm_W2.5mm_P5.00mm, F.Cu at (134.6, 134.6)
- added D1: LED, Connector_PinHeader_2.54mm:PinHeader_1x02_P2.54mm_Vertical, F.Cu at (127.0, 134.6)
- added J1: Screw_Terminal_01x02, TerminalBlock:TerminalBlock_Altech_AK300-2_P5.00mm, F.Cu at (101.6, 144.8)
- added Q1: Q_Photo_NPN, Connector_PinHeader_2.54mm:PinHeader_1x02_P2.54mm_Vertical, F.Cu at (127.0, 147.3)
- added R1: 43, Resistor_THT:R_Axial_DIN0204_L3.6mm_D1.6mm_P7.62mm_Horizontal, F.Cu at (116.8, 137.2)
- added R2: 22k, Resistor_THT:R_Axial_DIN0204_L3.6mm_D1.6mm_P7.62mm_Horizontal, F.Cu at (124.5, 142.2)
- added R3: 3k3, Resistor_THT:R_Axial_DIN0204_L3.6mm_D1.6mm_P7.62mm_Horizontal, F.Cu at (104.1, 139.7)
- added RV1: 10k, Potentiometer_THT:Potentiometer_ACP_CA9-H5_Horizontal, F.Cu at (146.1, 129.5)
- added U1: ESP1, Connector_PinHeader_2.54mm:PinHeader_2x04_P2.54mm_Vertical, F.Cu at (109.2, 132.1)
- added U2: MCP1700-3.3, Package_TO_SOT_THT:TO-92, F.Cu at (111.8, 147.3)
- added U3: LM293, Package_DIP:DIP-8_W7.62mm_Socket, F.Cu at (142.2, 139.7)
Routing:
- net VDD: track 0.00 -> 90.7 mm
- net GND: track 0.00 -> 88.9 mm
- net Net-(C1-Pad1): track 0.00 -> 35.3 mm
- net Net-(Q1-Pad2): track 0.00 -> 15.9 mm
- net VCC: track 0.00 -> 11.9 mm
- net Net-(R3-Pad2): track 0.00 -> 11.2 mm
- net Net-(RV1-Pad2): track 0.00 -> 6.75 mm
- net Net-(D1-Pad2): track 0.00 -> 2.54 mm

Commit message: additional elements and new board layout
Parts:
- added J2: Val, Connector_Pin:Pin_D0.7mm_L6.5mm_W1.8mm_FlatFork, F.Cu at (121.9, 147.3)
- added J3: Ref, Connector_Pin:Pin_D0.7mm_L6.5mm_W1.8mm_FlatFork, F.Cu at (147.3, 137.2)
- added J4: Gnd, Connector_Pin:Pin_D0.7mm_L6.5mm_W1.8mm_FlatFork, F.Cu at (129.5, 129.5)
- added R4: 3k3, Resistor_THT:R_Axial_DIN0204_L3.6mm_D1.6mm_P7.62mm_Horizontal, F.Cu at (152.4, 132.1)
- R1: value 43 -> 56
Connections:
- D1 pad 1: VDD -> Net-(D1-Pad1)
- D1 pad 2: Net-(D1-Pad2) -> VDD
- R1 pad 2: Net-(D1-Pad2) -> Net-(D1-Pad1)
- U3 pad 8: VDD -> VCC
Routing:
- net VCC: track 11.9 -> 42.7 mm
- net VDD: track 90.7 -> 80.2 mm
- net Net-(C1-Pad1): track 35.3 -> 45.5 mm
- net Net-(J2-Pad1): track 15.9 -> 22.0 mm
- net Net-(J3-Pad1): track 6.75 -> 11.6 mm
- net Net-(D1-Pad1): track 0.00 -> 3.59 mm
- net Net-(D1-Pad2): track 2.54 -> 0.00 mm

Commit message: pcb changes
Parts:
- moved D1 2.54 mm to (127.0, 137.2), turned to 180 degrees
Routing:
- net GND: track 88.9 -> 93.4 mm
- net Net-(J2-Pad1): track 22.0 -> 24.4 mm
- net Net-(D1-Pad1): track 3.59 -> 2.54 mm
- net VDD: track 80.2 -> 80.6 mm, vias 0 -> 1
Changed lines of the file:
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@@
-(kicad_pcb (version 20171130) (host pcbnew 5.1.4-e60b266~84~ubuntu16.04.1)
+(kicad_pcb (version 20171130) (host pcbnew 5.1.4)
   (general
     (thickness 1.6)
     (drawings 73)
-    (tracks 66)
+    (tracks 73)
     (zones 0)
     (modules 15)
@@
   )
   (module Connector_PinHeader_2.54mm:PinHeader_1x02_P2.54mm_Vertical (layer F.Cu)
-    (at 127 134.62)
+    (at 127 137.16 180)
     (descr "Through hole straight pin header, 1x02, 2.54mm pitch, single row")
     (tags "Through hole pin header THT 1x02 2.54mm single row")
@@
     (fp_line (start 1.27 -1.27) (end 1.27 3.81) (layer F.Fab) (width 0.1))
     (fp_line (start -0.635 -1.27) (end 1.27 -1.27) (layer F.Fab) (width 0.1))
-    (pad 2 thru_hole oval (at 0 2.54) (size 1.7 1.7) (drill 1) (layers *.Cu *.Mask)
+    (pad 2 thru_hole oval (at 0 2.54 180) (size 1.7 1.7) (drill 1) (layers *.Cu *.Mask)
       (net 3 VDD))
-    (pad 1 thru_hole rect (at 0 0) (size 1.7 1.7) (drill 1) (layers *.Cu *.Mask)
+    (pad 1 thru_hole rect (at 0 0 180) (size 1.7 1.7) (drill 1) (layers *.Cu *.Mask)
       (net 7 "Net-(D1-Pad1)"))
     (model ${KISYS3DMOD}/Connector_PinHeader_2.54mm.3dshapes/PinHeader_1x02_P2.54mm_Vertical.wrl
@@
   (segment (start 111.76 147.32) (end 116.84 142.24) (width 0.25) (layer F.Cu) (net 2))
   (segment (start 116.84 142.24) (end 116.84 137.16) (width 0.25) (layer F.Cu) (net 2))
-  (segment (start 111.76 132.08) (end 116.84 137.16) (width 0.25) (layer F.Cu) (net 2))
   (segment (start 135.745001 137.443629) (end 135.745001 130.745001) (width 0.25) (layer F.Cu) (net 2))
   (segment (start 134.62 138.56863) (end 135.745001 137.443629) (width 0.25) (layer F.Cu) (net 2))
@@
   (segment (start 135.745001 130.745001) (end 135.419999 130.419999) (width 0.25) (layer F.Cu) (net 2))
   (segment (start 134.62 139.7) (end 134.62 138.56863) (width 0.25) (layer F.Cu) (net 2))
+  (segment (start 110.12 144.78) (end 111.76 146.42) (width 0.25) (layer F.Cu) (net 2))
+  (segment (start 111.76 146.42) (end 111.76 147.32) (width 0.25) (layer F.Cu) (net 2))
+  (segment (start 101.6 144.78) (end 110.12 144.78) (width 0.25) (layer F.Cu) (net 2))
   (segment (start 112.679238 149.86) (end 111.76 149.86) (width 0.25) (layer F.Cu) (net 3))
   (segment (start 123.36 149.86) (end 112.679238 149.86) (width 0.25) (layer F.Cu) (net 3))
@@
   (segment (start 149.86 132.08) (end 148.59 132.08) (width 0.25) (layer F.Cu) (net 3))
   (segment (start 149.86 132.08) (end 152.4 132.08) (width 0.25) (layer F.Cu) (net 3))
-  (segment (start 143.51 132.08) (end 146.05 129.54) (width 0.25) (layer B.Cu) (net 3))
-  (segment (start 132.08 132.08) (end 143.51 132.08) (width 0.25) (layer B.Cu) (net 3))
-  (segment (start 127 137.16) (end 132.08 132.08) (width 0.25) (layer B.Cu) (net 3))
-  (segment (start 127 137.16) (end 127 138.43) (width 0.25) (layer F.Cu) (net 3))
-  (segment (start 127 138.43) (end 129.54 140.97) (width 0.25) (layer F.Cu) (net 3))
   (segment (start 128.1 147.32) (end 127 147.32) (width 0.25) (layer F.Cu) (net 3))
   (segment (start 129.54 145.88) (end 128.1 147.32) (width 0.25) (layer F.Cu) (net 3))
   (segment (start 129.54 140.97) (end 129.54 145.88) (width 0.25) (layer F.Cu) (net 3))
-  (segment (start 124.46 142.24) (end 127 144.78) (width 0.25) (layer B.Cu) (net 8))
-  (segment (start 132.08 144.78) (end 127 144.78) (width 0.25) (layer B.Cu) (net 8))
-  (segment (start 137.16 139.7) (end 132.08 144.78) (width 0.25) (layer B.Cu) (net 8))
+  (segment (start 129.54 140.97) (end 129.54 134.62) (width 0.25) (layer F.Cu) (net 3))
+  (segment (start 127 134.62) (end 129.54 134.62) (width 0.25) (layer F.Cu) (net 3))
+  (via (at 129.54 134.62) (size 0.8) (drill 0.4) (layers F.Cu B.Cu) (net 3))
+  (segment (start 144.880001 130.709999) (end 146.05 129.54) (width 0.25) (layer B.Cu) (net 3))
+  (segment (start 142.24 133.35) (end 144.880001 130.709999) (width 0.25) (layer B.Cu) (net 3))
+  (segment (start 130.81 133.35) (end 142.24 133.35) (width 0.25) (layer B.Cu) (net 3))
+  (segment (start 129.54 134.62) (end 130.81 133.35) (width 0.25) (layer B.Cu) (net 3))
   (segment (start 110.910001 133.770001) (end 111.76 134.62) (width 0.25) (layer F.Cu) (net 4))
   (segment (start 110.584999 133.444999) (end 110.910001 133.770001) (width 0.25) (layer F.Cu) (net 4))
@@
   (segment (start 104.14 132.08) (end 105.504999 133.444999) (width 0.25) (layer F.Cu) (net 4))
   (segment (start 111.76 137.16) (end 111.76 134.62) (width 0.25) (layer F.Cu) (net 4))
-  (segment (start 139.7 138.39) (end 139.7 139.7) (width 0.25) (layer F.Cu) (net 9))
-  (segment (start 143.55 134.54) (end 139.7 138.39) (width 0.25) (layer F.Cu) (net 9))
   (segment (start 112.110762 148.59) (end 113.03 148.59) (width 0.25) (layer F.Cu) (net 6))
   (segment (start 111.586998 148.59) (end 112.110762 148.59) (width 0.25) (layer F.Cu) (net 6))
@@
   (segment (start 139.7 149.86) (end 142.24 147.32) (width 0.25) (layer B.Cu) (net 6))
   (segment (start 132.08 149.86) (end 139.7 149.86) (width 0.25) (layer B.Cu) (net 6))
-  (segment (start 124.46 137.16) (end 127 134.62) (width 0.25) (layer B.Cu) (net 7))
+  (segment (start 127 137.16) (end 124.46 137.16) (width 0.25) (layer B.Cu) (net 7))
+  (segment (start 124.46 142.24) (end 127 144.78) (width 0.25) (layer B.Cu) (net 8))
   (segment (start 121.92 144.78) (end 124.46 142.24) (width 0.25) (layer B.Cu) (net 8))
   (segment (start 121.92 147.32) (end 121.92 144.78) (width 0.25) (layer B.Cu) (net 8))
+  (segment (start 131.301411 138.574999) (end 127.63641 142.24) (width 0.25) (layer B.Cu) (net 8))
+  (segment (start 125.449949 142.24) (end 124.46 142.24) (width 0.25) (layer B.Cu) (net 8))
+  (segment (start 127.63641 142.24) (end 125.449949 142.24) (width 0.25) (layer B.Cu) (net 8))
+  (segment (start 136.034999 138.574999) (end 131.301411 138.574999) (width 0.25) (layer B.Cu) (net 8))
+  (segment (start 137.16 139.7) (end 136.034999 138.574999) (width 0.25) (layer B.Cu) (net 8))
+  (segment (start 139.7 138.39) (end 139.7 139.7) (width 0.25) (layer F.Cu) (net 9))
+  (segment (start 143.55 134.54) (end 139.7 138.39) (width 0.25) (layer F.Cu) (net 9))
   (segment (start 146.17 137.16) (end 143.55 134.54) (width 0.25) (layer F.Cu) (net 9))
   (segment (start 147.32 137.16) (end 146.17 137.16) (width 0.25) (layer F.Cu) (net 9))
